File: 10AxisFeatherWingLE.brd (EAGLE design)
At the start: 50.8 x 22.9 mm, 17 parts, among them IC1 LSM9DS1, U2 BME280

Commit message: Added new features
Added breakouts and silk text.
Parts:
- removed R4: 10K, microbuilder:0603-NO
- added JP2: (no value), microbuilder:1X05_ROUND_70
- added R2: 10K, microbuilder:0603-NO
- C3: value 10nF -> 0.1uF
- C4: value 0.1uF -> 10nF
- moved R3 26.7 mm to (17.8, 12.7), turned to 270 degrees
- moved U2 24.1 mm to (12.7, 11.4)
- moved SJ1 21.9 mm to (9.84, 9.53), turned to 90 degrees
- moved R1 19.1 mm to (12.7, 8.89), turned to 0 degrees
- moved C1 12.5 mm to (21.0, 8.89), turned to 90 degrees
- moved C5 10.6 mm to (10.2, 13.3), turned to 270 degrees
- moved C4 8.89 mm to (22.9, 12.7), turned to 270 degrees
- moved C6 7.41 mm to (12.7, 14.0), turned to 180 degrees
- moved C2 5.39 mm to (22.9, 8.89), turned to 90 degrees
- moved C3 3.17 mm to (21.0, 12.7), turned to 270 degrees
Connections:
- new net DEN_A/G: IC1.13, JP2.5
- new net DRDY_M: IC1.9, JP2.1
- new net INT1_A/G: IC1.11, JP2.3
- new net INT2_A/G: IC1.12, JP2.4
- new net INT_M: IC1.10, JP2.2
- net 3.3V: now also C3.2, R2.1; no longer C4.2, IC1.5, IC1.6, R4.1
- net CAP: now also C4.2; no longer C3.2
- net GND: now also IC1.5, IC1.6
- net SCL: now also R2.2; no longer R4.2
Routing:
- net 3.3V: track 94.3 -> 63.9 mm
- net DRDY_M: track 0.00 -> 23.4 mm
- net DEN_A/G: track 0.00 -> 23.4 mm
- net INT_M: track 0.00 -> 22.5 mm
- net INT2_A/G: track 0.00 -> 22.5 mm
- net INT1_A/G: track 0.00 -> 21.6 mm
- net GND: track 19.1 -> 28.9 mm, vias 10 -> 4
- net SCL: track 47.5 -> 40.9 mm, vias 3 -> 2
- net CAP: track 5.77 -> 1.40 mm
- net C1: track 5.25 -> 1.57 mm
- net SDO: track 5.75 -> 3.53 mm
- net SDA: track 47.6 -> 49.1 mm, vias 1 -> 2
- net RESET: track 2.54 -> 3.44 mm
Other:
- board text added: "(C) Mark Aldritz Dela Virgen"
- board text added: "10AxisFeatherWingLE"
- board text added: "DEN"
- board text added: "DRDY"
- board text added: "I2C ADDR"
- board text added: "INT1"
- board text added: "INT2"
- board text added: "INTM"
- board text added: "Simple I2C 10-DOF FeatherWing"
