File: 10AxisFeatherWingLE.sch (EAGLE design)
At the start: 17 parts, among them IC1 LSM9DS1, U2 BME280

Commit message: Added new features
Added breakouts and silk text.
Parts:
- removed R4: 10K, microbuilder:RESISTOR_0603_NOOUT
- added JP2: (no value), microbuilder:HEADER-1X570MIL
- added R2: 10K, microbuilder:RESISTOR_0603_NOOUT
- C3: value 10nF -> 0.1uF
- C4: value 0.1uF -> 10nF
Connections:
- new net DEN_A/G: IC1.DEN_A/G, JP2.5
- new net DRDY_M: IC1.DRDY_M, JP2.1
- new net INT1_A/G: IC1.INT1_A/G, JP2.3
- new net INT2_A/G: IC1.INT2_A/G, JP2.4
- new net INT_M: IC1.INT_M, JP2.2
- net 3.3V: now also C3.2, R2.1; no longer C4.2, IC1.SDO_A/G, IC1.SDO_M, R4.1
- net CAP: now also C4.2; no longer C3.2
- net GND: now also IC1.SDO_A/G, IC1.SDO_M
- net SCL: now also R2.2; no longer R4.2
Other:
- moved on the sheet: C1, C3, C4, C5, C6, R3
